Commit message: Add parameters for actuator configuration
Signed-off-by: Victor T. N <victortn21@hotmail.com>

File: description/ic2d.urdf.xacro (robot description, xacro)
@@ -1,4 +1,12 @@
 <?xml version="1.0"?>
 <robot xmlns:xacro="http://www.ros.org/wiki/xacro" name="ic2d">
+    <!-- Joint configurations:
+         "linmot": LinMot P01-37x120F/40x120-HP
+         "hydraulic": Hoerbiger LB6161000804M
+         "fixed": no motion -->
+    <xacro:arg name="joint_1_config" default="linmot"/>
+    <xacro:arg name="joint_2_config" default="linmot"/>
+    <xacro:property name="joint_1_config" value="$(arg joint_1_config)"/>
+    <xacro:property name="joint_2_config" value="$(arg joint_2_config)"/>
     <xacro:include filename="ic2d_core.xacro"/>
     <xacro:include filename="ros2_control.xacro"/>

File: description/ic2d_core.xacro (robot description, xacro)
@@ -2,4 +2,5 @@
 <robot xmlns:xacro="http://www.ros.org/wiki/xacro">
     <xacro:include filename="ic2d_materials.xacro"/>
+    <xacro:include filename="ic2d_actuators.xacro"/>
     <link name="world"/>
     <link name="base_link">
@@ -48,11 +49,31 @@
     </collision>
   </link>
-  <joint name="joint_1" type="prismatic">
-    <origin xyz="-0.088092 0 0.18042" rpy="0 0 0" />
-    <parent link="base_link" />
-    <child link="link_1" />
-    <axis xyz="1 0 0" />
-    <limit lower="0" upper="0.5" effort="1000" velocity="100" />
-  </joint>
+  <xacro:if value="${joint_1_config == 'linmot'}">
+    <joint name="joint_1" type="prismatic">
+      <origin xyz="-0.088092 0 0.18042" rpy="0 0 0" />
+      <parent link="base_link" />
+      <child link="link_1" />
+      <axis xyz="1 0 0" />
+      <limit lower="0" upper="${linmot_stroke}" effort="${linmot_effort}" velocity="${linmot_velocity}" />
+    </joint>
+  </xacro:if>
+  <xacro:if value="${joint_1_config == 'hydraulic'}">
+    <joint name="joint_1" type="prismatic">
+      <origin xyz="-0.088092 0 0.18042" rpy="0 0 0" />
+      <parent link="base_link" />
+      <child link="link_1" />
+      <axis xyz="1 0 0" />
+      <limit lower="0" upper="${hydraulic_stroke}" effort="${hydraulic_effort}" velocity="${hydraulic_velocity}" />
+    </joint>
+  </xacro:if>
+  <xacro:if value="${joint_1_config == 'fixed'}">
+    <joint name="joint_1" type="prismatic">
+      <origin xyz="-0.088092 0 0.18042" rpy="0 0 0" />
+      <parent link="base_link" />
+      <child link="link_1" />
+      <axis xyz="1 0 0" />
+      <limit lower="0" upper="0" effort="9999999999999" velocity="0" />
+    </joint>
+  </xacro:if>
   <link name="link_2">
     <inertial>
@@ -75,10 +96,30 @@
     </collision>
   </link>
-  <joint name="joint_2" type="prismatic">
-    <origin xyz="0.35443 0 0.18042" rpy="0 0 0" />
-    <parent link="base_link" />
-    <child link="link_2" />
-    <axis xyz="1 0 0" />
-    <limit lower="-0.5" upper="0" effort="1000" velocity="100" />
-  </joint>
+  <xacro:if value="${joint_2_config == 'linmot'}">
+    <joint name="joint_2" type="prismatic">
+      <origin xyz="0.35443 0 0.18042" rpy="0 0 0" />
+      <parent link="base_link" />
+      <child link="link_2" />
+      <axis xyz="1 0 0" />
+      <limit lower="-${linmot_stroke}" upper="0" effort="${linmot_effort}" velocity="${linmot_velocity}" />
+    </joint>
+  </xacro:if>
+  <xacro:if value="${joint_2_config == 'hydraulic'}">
+    <joint name="joint_2" type="prismatic">
+      <origin xyz="0.35443 0 0.18042" rpy="0 0 0" />
+      <parent link="base_link" />
+      <child link="link_2" />
+      <axis xyz="1 0 0" />
+      <limit lower="-${hydraulic_stroke}" upper="0" effort="${hydraulic_effort}" velocity="${hydraulic_velocity}" />
+    </joint>
+  </xacro:if>
+  <xacro:if value="${joint_2_config == 'fixed'}">
+    <joint name="joint_2" type="prismatic">
+      <origin xyz="0.35443 0 0.18042" rpy="0 0 0" />
+      <parent link="base_link" />
+      <child link="link_2" />
+      <axis xyz="1 0 0" />
+      <limit lower="0" upper="0" effort="9999999999999" velocity="0" />
+    </joint>
+  </xacro:if>
 </robot>

File: description/ros2_control.xacro (robot description, xacro)
@@ -8,5 +8,13 @@
             <command_interface name="position">
                 <param name="min">0</param>
-                <param name="max">0.5</param>
+                <xacro:if value="${joint_1_config == 'linmot'}">
+                    <param name="max">${linmot_stroke}</param>
+                </xacro:if>
+                <xacro:if value="${joint_1_config == 'hydraulic'}">
+                    <param name="max">${hydraulic_stroke}</param>
+                </xacro:if>
+                <xacro:if value="${joint_1_config == 'fixed'}">
+                    <param name="max">0</param>
+                </xacro:if>
             </command_interface>
             <state_interface name="position"/>
@@ -16,5 +24,13 @@
         <joint name="joint_2">
             <command_interface name="position">
-                <param name="min">-0.5</param>
+                <xacro:if value="${joint_2_config == 'linmot'}">
+                    <param name="min">-${linmot_stroke}</param>
+                </xacro:if>
+                <xacro:if value="${joint_2_config == 'hydraulic'}">
+                    <param name="min">-${hydraulic_stroke}</param>
+                </xacro:if>
+                <xacro:if value="${joint_2_config == 'fixed'}">
+                    <param name="min">0</param>
+                </xacro:if>
                 <param name="max">0</param>
             </command_interface>

Commit message: Add parameters for customizing link masses
Signed-off-by: Victor T. N <victortn21@hotmail.com>

File: description/ic2d.urdf.xacro (robot description, xacro)
@@ -7,6 +7,11 @@
     <xacro:arg name="joint_1_config" default="linmot"/>
     <xacro:arg name="joint_2_config" default="linmot"/>
+    <xacro:arg name="link_1_mass" default="18.505"/>
+    <xacro:arg name="link_2_mass" default="7.3822"/>
+    <!-- Convert args to properties for easier syntax -->
     <xacro:property name="joint_1_config" value="$(arg joint_1_config)"/>
     <xacro:property name="joint_2_config" value="$(arg joint_2_config)"/>
+    <xacro:property name="link_1_mass" value="$(arg link_1_mass)"/>
+    <xacro:property name="link_2_mass" value="$(arg link_2_mass)"/>
     <xacro:include filename="ic2d_core.xacro"/>
     <xacro:include filename="ros2_control.xacro"/>

File: description/ic2d_core.xacro (robot description, xacro)
@@ -3,4 +3,5 @@
     <xacro:include filename="ic2d_materials.xacro"/>
     <xacro:include filename="ic2d_actuators.xacro"/>
+    <xacro:include filename="inertial_macros.xacro"/>
     <link name="world"/>
     <link name="base_link">
@@ -30,9 +31,14 @@
   </joint>
   <link name="link_1">
+    <!-- CAD-generated inertial block
     <inertial>
       <origin xyz="-0.20394 5.3438E-06 -0.015363" rpy="0 0 0" />
       <mass value="18.505" />
       <inertia ixx="0.12026" ixy="9.5669E-07" ixz="-3.1152E-06" iyy="0.014885" iyz="-6.6837E-08" izz="0.12951" />
-    </inertial>
+    </inertial> -->
+    <xacro:inertial_box mass="${link_1_mass}" x="0.378020" y="0.315000" z="0.159020">
+      <!-- Macro inertial block. XYZ dimensions correspond to link_1.STL bounding box -->
+      <origin xyz="-0.20394 5.3438E-06 -0.015363" rpy="0 0 0" />
+    </xacro:inertial_box>
     <visual>
       <origin xyz="0 0 0" rpy="0 0 0" />
@@ -77,9 +83,14 @@
   </xacro:if>
   <link name="link_2">
+    <!-- CAD-generated inertial block
     <inertial>
       <origin xyz="0.063069 -1.9306E-06 -0.02353" rpy="0 0 0" />
       <mass value="7.3822" />
       <inertia ixx="0.044429" ixy="2.1429E-07" ixz="4.9245E-07" iyy="0.0054955" iyz="6.0516E-08" izz="0.047349" />
-    </inertial>
+    </inertial> -->
+    <xacro:inertial_box mass="${link_2_mass}" x="0.119020" y="0.315000" z="0.099020">
+      <!-- Macro inertial block. XYZ dimensions correspond to link_2.STL bounding box -->
+      <origin xyz="0.063069 -1.9306E-06 -0.02353" rpy="0 0 0" />
+    </xacro:inertial_box>
     <visual>
       <origin xyz="0 0 0" rpy="0 0 0" />
